File: Eagle Files/RAMPSDC.sch (EAGLE design)
At the start: 20 parts, among them IC1 AT24CP, IC2 7805T, U1 ARDUINO_MEGA_SHIELD

Commit message: Disconnected Max Endstops and Servos 2-4. Added SD card Headers. Fixed some Silkscreen errors.
This is a step towards making the LCD screen work, but in the meantime,
the last level shifter was changed to all NC. At some point, that will
be the encoder button, encoder 1, encoder 2, MISO, and whatever else
needs to be shifted to make the reprap full graphics controller work.
The issue is the documentation sucks on that so I need to really dig to
make it work. In the meantime, I added just a breakout header for the
generic 6-pin SD card module for arduinos. This doesnt replace an LCD,
but at least makes it run standalone.

The Max Endstops were not rerouted to anywhere, and are disconnected
from the rest of the system to prevent someone accidently frying their
Due. The Servo pins are outputs, so they were connected back the their
respective pins, but are not level shifted, so they may behave
strangely. The first Servo pin (SERVO0) is level shifted.
Parts:
- removed JP6: (no value), adafruit:PINHD-1X6
- added JP9: (no value), adafruit:PINHD-1X6
Connections:
- removed net +5V: ARDUINO_DUE1.5V_SPI, JP6.2
- removed net LV_D11: ARDUINO_DUE1.11, JP1.1
- removed net LV_D5: ARDUINO_DUE1.5, JP1.5
- removed net LV_D6: ARDUINO_DUE1.6, JP1.2
- new net N$10: JP3.6
- new net N$11: JP4.6
- new net N$2: JP1.1
- new net N$3: JP1.2
- new net N$4: JP2.1
- new net N$5: JP2.2
- new net N$6: JP2.5
- new net N$7: JP2.6
- new net N$8: JP1.6
- new net N$9: JP1.5
- net +3.3V: now also JP5.3, JP9.1, JP9.5
- net CANRX: no longer JP5.3
- net CANTX: no longer JP5.4
- net D11: now also ARDUINO_DUE1.11; no longer JP2.1
- net D4: now also JP8.6; no longer JP2.6
- net D5: now also ARDUINO_DUE1.5; no longer JP2.5
- net D6: now also ARDUINO_DUE1.6; no longer JP2.2
- net GND: now also JP5.4, JP9.6; no longer JP6.6
- net LV_D4: now also JP7.6; no longer JP1.6
- net LV_X-MAX: no longer JP7.6
- net LV_Y-MAX: no longer JP3.6
- net MASTER_R: no longer JP6.5
- net MISO: now also JP9.4; no longer JP6.1
- net MOSI: now also JP9.3; no longer JP6.4
- net SPCK: now also JP9.2; no longer JP6.3
- net X-MAX: no longer JP8.6
- net Y-MAX: no longer JP4.6
Other:
- note added: "SD Card AUX"
